Commit message: update to the latest alrobotmodelutils

File: pepper_description/urdf/pepper1.0_generated_urdf/pepper_arms.xacro (robot description, xacro)
@@ -86,5 +86,10 @@
 		<limit effort="0.144" lower="0.02" upper="0.98" velocity="12.56"/>
 	</joint>
-	<link name="l_gripper"/>
+	<link name="l_gripper">
+		<inertial>
+			<mass value="2e-06"/>
+			<inertia ixx="1.1e-09" ixy="0" ixz="0" iyy="1.1e-09" iyz="0" izz="1.1e-09"/>
+		</inertial>
+	</link>
 	<joint name="RShoulderPitch" type="revolute">
 		<parent link="torso"/>
@@ -169,4 +174,9 @@
 		<limit effort="0.144" lower="0.02" upper="0.98" velocity="12.56"/>
 	</joint>
-	<link name="r_gripper"/>
+	<link name="r_gripper">
+		<inertial>
+			<mass value="2e-06"/>
+			<inertia ixx="1.1e-09" ixy="0" ixz="0" iyy="1.1e-09" iyz="0" izz="1.1e-09"/>
+		</inertial>
+	</link>
 </robot>

File: pepper_description/urdf/pepper1.0_generated_urdf/pepper_fingers.xacro (robot description, xacro)
@@ -3,6 +3,10 @@
  ****** File automatically generated by generate_urdf.py script ******
  *********************************************************************-->
-<robot name="julietteY20MP" xmlns:xacro="http://www.ros.org/wiki/xacro">
+<robot name="JulietteY20MP" xmlns:xacro="http://www.ros.org/wiki/xacro">
 	<link name="RFinger41_link">
+		<inertial>
+			<mass value="2e-06"/>
+			<inertia ixx="1.1e-09" ixy="0" ixz="0" iyy="1.1e-09" iyz="0" izz="1.1e-09"/>
+		</inertial>
 		<xacro:insert_visu_RFinger41_link/>
 	</link>
@@ -15,4 +19,8 @@
 	</joint>
 	<link name="LFinger42_link">
+		<inertial>
+			<mass value="2e-06"/>
+			<inertia ixx="1.1e-09" ixy="0" ixz="0" iyy="1.1e-09" iyz="0" izz="1.1e-09"/>
+		</inertial>
 		<xacro:insert_visu_LFinger42_link/>
 	</link>
@@ -25,4 +33,8 @@
 	</joint>
 	<link name="RFinger11_link">
+		<inertial>
+			<mass value="2e-06"/>
+			<inertia ixx="1.1e-09" ixy="0" ixz="0" iyy="1.1e-09" iyz="0" izz="1.1e-09"/>
+		</inertial>
 		<xacro:insert_visu_RFinger11_link/>
 	</link>
@@ -35,4 +47,8 @@
 	</joint>
 	<link name="RFinger12_link">
+		<inertial>
+			<mass value="2e-06"/>
+			<inertia ixx="1.1e-09" ixy="0" ixz="0" iyy="1.1e-09" iyz="0" izz="1.1e-09"/>
+		</inertial>
 		<xacro:insert_visu_RFinger12_link/>
 	</link>
@@ -45,4 +61,8 @@
 	</joint>
 	<link name="LFinger33_link">
+		<inertial>
+			<mass value="2e-06"/>
+			<inertia ixx="1.1e-09" ixy="0" ixz="0" iyy="1.1e-09" iyz="0" izz="1.1e-09"/>
+		</inertial>
 		<xacro:insert_visu_LFinger33_link/>
 	</link>
@@ -54,5 +74,37 @@
 		<mimic joint="LHand" multiplier="0.872665" offset="0"/>
 	</joint>
+	<link name="RFinger31_link">
+		<inertial>
+			<mass value="2e-06"/>
+			<inertia ixx="1.1e-09" ixy="0" ixz="0" iyy="1.1e-09" iyz="0" izz="1.1e-09"/>
+		</inertial>
+		<xacro:insert_visu_RFinger31_link/>
+	</link>
+	<joint name="RFinger31" type="continuous">
+		<parent link="r_wrist"/>
+		<child link="RFinger31_link"/>
+		<origin rpy="1.67523 1.04483 0.029316" xyz="0.0833 -0.0123 0.004"/>
+		<axis xyz="0 0 1.0"/>
+		<mimic joint="RHand" multiplier="0.872665" offset="0"/>
+	</joint>
+	<link name="LFinger21_link">
+		<inertial>
+			<mass value="2e-06"/>
+			<inertia ixx="1.1e-09" ixy="0" ixz="0" iyy="1.1e-09" iyz="0" izz="1.1e-09"/>
+		</inertial>
+		<xacro:insert_visu_LFinger21_link/>
+	</link>
+	<joint name="LFinger21" type="continuous">
+		<parent link="l_wrist"/>
+		<child link="LFinger21_link"/>
+		<origin rpy="1.5708 1.0472 -0.061086" xyz="0.0873 -0.0073 0.006"/>
+		<axis xyz="0 0 1.0"/>
+		<mimic joint="LHand" multiplier="0.872665" offset="0"/>
+	</joint>
 	<link name="RFinger32_link">
+		<inertial>
+			<mass value="2e-06"/>
+			<inertia ixx="1.1e-09" ixy="0" ixz="0" iyy="1.1e-09" iyz="0" izz="1.1e-09"/>
+		</inertial>
 		<xacro:insert_visu_RFinger32_link/>
 	</link>
@@ -64,15 +116,177 @@
 		<mimic joint="RHand" multiplier="0.872665" offset="0"/>
 	</joint>
-	<link name="LFinger21_link">
-		<xacro:insert_visu_LFinger21_link/>
-	</link>
-	<joint name="LFinger21" type="continuous">
-		<parent link="l_wrist"/>
-		<child link="LFinger21_link"/>
-		<origin rpy="1.5708 1.0472 -0.061086" xyz="0.0873 -0.0073 0.006"/>
+	<link name="LFinger13_link">
+		<inertial>
+			<mass value="2e-06"/>
+			<inertia ixx="1.1e-09" ixy="0" ixz="0" iyy="1.1e-09" iyz="0" izz="1.1e-09"/>
+		</inertial>
+		<xacro:insert_visu_LFinger13_link/>
+	</link>
+	<joint name="LFinger13" type="continuous">
+		<parent link="LFinger12_link"/>
+		<child link="LFinger13_link"/>
+		<origin rpy="0 0 -1.0472" xyz="0.018 0 0"/>
+		<axis xyz="0 0 1.0"/>
+		<mimic joint="LHand" multiplier="0.872665" offset="0"/>
+	</joint>
+	<link name="LFinger32_link">
+		<inertial>
+			<mass value="2e-06"/>
+			<inertia ixx="1.1e-09" ixy="0" ixz="0" iyy="1.1e-09" iyz="0" izz="1.1e-09"/>
+		</inertial>
+		<xacro:insert_visu_LFinger32_link/>
+	</link>
+	<joint name="LFinger32" type="continuous">
+		<parent link="LFinger31_link"/>
+		<child link="LFinger32_link"/>
+		<origin rpy="0 0 -1.0472" xyz="0.018 0 0"/>
+		<axis xyz="0 0 1.0"/>
+		<mimic joint="LHand" multiplier="0.872665" offset="0"/>
+	</joint>
+	<link name="LFinger11_link">
+		<inertial>
+			<mass value="2e-06"/>
+			<inertia ixx="1.1e-09" ixy="0" ixz="0" iyy="1.1e-09" iyz="0" izz="1.1e-09"/>
+		</inertial>
+		<xacro:insert_visu_LFinger11_link/>
+	</link>
+	<joint name="LFinger11" type="continuous">
+		<parent link="l_wrist"/>
+		<child link="LFinger11_link"/>
+		<origin rpy="1.74402 1.04064 -0.0334335" xyz="0.0821 -0.0268 0.004"/>
+		<axis xyz="0 0 1.0"/>
+		<mimic joint="LHand" multiplier="0.872665" offset="0"/>
+	</joint>
+	<link name="RFinger22_link">
+		<inertial>
+			<mass value="2e-06"/>
+			<inertia ixx="1.1e-09" ixy="0" ixz="0" iyy="1.1e-09" iyz="0" izz="1.1e-09"/>
+		</inertial>
+		<xacro:insert_visu_RFinger22_link/>
+	</link>
+	<joint name="RFinger22" type="continuous">
+		<parent link="RFinger21_link"/>
+		<child link="RFinger22_link"/>
+		<origin rpy="0 0 -1.0472" xyz="0.018 0 0"/>
+		<axis xyz="0 0 1.0"/>
+		<mimic joint="RHand" multiplier="0.872665" offset="0"/>
+	</joint>
+	<link name="RFinger13_link">
+		<inertial>
+			<mass value="2e-06"/>
+			<inertia ixx="1.1e-09" ixy="0" ixz="0" iyy="1.1e-09" iyz="0" izz="1.1e-09"/>
+		</inertial>
+		<xacro:insert_visu_RFinger13_link/>
+	</link>
+	<joint name="RFinger13" type="continuous">
+		<parent link="RFinger12_link"/>
+		<child link="RFinger13_link"/>
+		<origin rpy="0 0 -1.0472" xyz="0.018 0 0"/>
+		<axis xyz="0 0 1.0"/>
+		<mimic joint="RHand" multiplier="0.872665" offset="0"/>
+	</joint>
+	<link name="LFinger22_link">
+		<inertial>
+			<mass value="2e-06"/>
+			<inertia ixx="1.1e-09" ixy="0" ixz="0" iyy="1.1e-09" iyz="0" izz="1.1e-09"/>
+		</inertial>
+		<xacro:insert_visu_LFinger22_link/>
+	</link>
+	<joint name="LFinger22" type="continuous">
+		<parent link="LFinger21_link"/>
+		<child link="LFinger22_link"/>
+		<origin rpy="0 0 -1.0472" xyz="0.018 0 0"/>
+		<axis xyz="0 0 1.0"/>
+		<mimic joint="LHand" multiplier="0.872665" offset="0"/>
+	</joint>
+	<link name="RFinger21_link">
+		<inertial>
+			<mass value="2e-06"/>
+			<inertia ixx="1.1e-09" ixy="0" ixz="0" iyy="1.1e-09" iyz="0" izz="1.1e-09"/>
+		</inertial>
+		<xacro:insert_visu_RFinger21_link/>
+	</link>
+	<joint name="RFinger21" type="continuous">
+		<parent link="r_wrist"/>
+		<child link="RFinger21_link"/>
+		<origin rpy="1.5708 1.0472 0.061086" xyz="0.0873 0.0073 0.006"/>
+		<axis xyz="0 0 1.0"/>
+		<mimic joint="RHand" multiplier="0.872665" offset="0"/>
+	</joint>
+	<link name="LFinger41_link">
+		<inertial>
+			<mass value="2e-06"/>
+			<inertia ixx="1.1e-09" ixy="0" ixz="0" iyy="1.1e-09" iyz="0" izz="1.1e-09"/>
+		</inertial>
+		<xacro:insert_visu_LFinger41_link/>
+	</link>
+	<joint name="LFinger41" type="continuous">
+		<parent link="l_wrist"/>
+		<child link="LFinger41_link"/>
+		<origin rpy="1.39757 1.04064 0.0683394" xyz="0.074 0.0309 0"/>
+		<axis xyz="0 0 1.0"/>
+		<mimic joint="LHand" multiplier="0.872665" offset="0"/>
+	</joint>
+	<link name="LFinger12_link">
+		<inertial>
+			<mass value="2e-06"/>
+			<inertia ixx="1.1e-09" ixy="0" ixz="0" iyy="1.1e-09" iyz="0" izz="1.1e-09"/>
+		</inertial>
+		<xacro:insert_visu_LFinger12_link/>
+	</link>
+	<joint name="LFinger12" type="continuous">
+		<parent link="LFinger11_link"/>
+		<child link="LFinger12_link"/>
+		<origin rpy="0 0 -1.0472" xyz="0.018 0 0"/>
+		<axis xyz="0 0 1.0"/>
+		<mimic joint="LHand" multiplier="0.872665" offset="0"/>
+	</joint>
+	<link name="RFinger23_link">
+		<inertial>
+			<mass value="2e-06"/>
+			<inertia ixx="1.1e-09" ixy="0" ixz="0" iyy="1.1e-09" iyz="0" izz="1.1e-09"/>
+		</inertial>
+		<xacro:insert_visu_RFinger23_link/>
+	</link>
+	<joint name="RFinger23" type="continuous">
+		<parent link="RFinger22_link"/>
+		<child link="RFinger23_link"/>
+		<origin rpy="0 0 -1.0472" xyz="0.018 0 0"/>
+		<axis xyz="0 0 1.0"/>
+		<mimic joint="RHand" multiplier="0.872665" offset="0"/>
+	</joint>
+	<link name="LFinger23_link">
+		<inertial>
+			<mass value="2e-06"/>
+			<inertia ixx="1.1e-09" ixy="0" ixz="0" iyy="1.1e-09" iyz="0" izz="1.1e-09"/>
+		</inertial>
+		<xacro:insert_visu_LFinger23_link/>
+	</link>
+	<joint name="LFinger23" type="continuous">
+		<parent link="LFinger22_link"/>
+		<child link="LFinger23_link"/>
+		<origin rpy="0 0 -1.0472" xyz="0.018 0 0"/>
+		<axis xyz="0 0 1.0"/>
+		<mimic joint="LHand" multiplier="0.872665" offset="0"/>
+	</joint>
+	<link name="LFinger43_link">
+		<inertial>
+			<mass value="2e-06"/>
+			<inertia ixx="1.1e-09" ixy="0" ixz="0" iyy="1.1e-09" iyz="0" izz="1.1e-09"/>
+		</inertial>
+		<xacro:insert_visu_LFinger43_link/>
+	</link>
+	<joint name="LFinger43" type="continuous">
+		<parent link="LFinger42_link"/>
+		<child link="LFinger43_link"/>
+		<origin rpy="0 0 -1.0472" xyz="0.018 0 0"/>
 		<axis xyz="0 0 1.0"/>
 		<mimic joint="LHand" multiplier="0.872665" offset="0"/>
 	</joint>
 	<link name="RFinger43_link">
+		<inertial>
+			<mass value="2e-06"/>
+			<inertia ixx="1.1e-09" ixy="0" ixz="0" iyy="1.1e-09" iyz="0" izz="1.1e-09"/>
+		</inertial>
 		<xacro:insert_visu_RFinger43_link/>
 	</link>
@@ -84,125 +298,9 @@
 		<mimic joint="RHand" multiplier="0.872665" offset="0"/>
 	</joint>
-	<link name="LFinger13_link">
-		<xacro:insert_visu_LFinger13_link/>
-	</link>
-	<joint name="LFinger13" type="continuous">
-		<parent link="LFinger12_link"/>
-		<child link="LFinger13_link"/>
-		<origin rpy="0 0 -1.0472" xyz="0.018 0 0"/>
-		<axis xyz="0 0 1.0"/>
-		<mimic joint="LHand" multiplier="0.872665" offset="0"/>
-	</joint>
-	<link name="LFinger32_link">
-		<xacro:insert_visu_LFinger32_link/>
-	</link>
-	<joint name="LFinger32" type="continuous">
-		<parent link="LFinger31_link"/>
-		<child link="LFinger32_link"/>
-		<origin rpy="0 0 -1.0472" xyz="0.018 0 0"/>
-		<axis xyz="0 0 1.0"/>
-		<mimic joint="LHand" multiplier="0.872665" offset="0"/>
-	</joint>
-	<link name="LFinger11_link">
-		<xacro:insert_visu_LFinger11_link/>
-	</link>
-	<joint name="LFinger11" type="continuous">
-		<parent link="l_wrist"/>
-		<child link="LFinger11_link"/>
-		<origin rpy="1.74402 1.04064 -0.0334335" xyz="0.0821 -0.0268 0.004"/>
-		<axis xyz="0 0 1.0"/>
-		<mimic joint="LHand" multiplier="0.872665" offset="0"/>
-	</joint>
-	<link name="RFinger22_link">
-		<xacro:insert_visu_RFinger22_link/>
-	</link>
-	<joint name="RFinger22" type="continuous">
-		<parent link="RFinger21_link"/>
-		<child link="RFinger22_link"/>
-		<origin rpy="0 0 -1.0472" xyz="0.018 0 0"/>
-		<axis xyz="0 0 1.0"/>
-		<mimic joint="RHand" multiplier="0.872665" offset="0"/>
-	</joint>
-	<link name="LFinger41_link">
-		<xacro:insert_visu_LFinger41_link/>
-	</link>
-	<joint name="LFinger41" type="continuous">
-		<parent link="l_wrist"/>
-		<child link="LFinger41_link"/>
-		<origin rpy="1.39757 1.04064 0.0683394" xyz="0.074 0.0309 0"/>
-		<axis xyz="0 0 1.0"/>
-		<mimic joint="LHand" multiplier="0.872665" offset="0"/>
-	</joint>
-	<link name="RFinger13_link">
-		<xacro:insert_visu_RFinger13_link/>
-	</link>
-	<joint name="RFinger13" type="continuous">
-		<parent link="RFinger12_link"/>
-		<child link="RFinger13_link"/>
-		<origin rpy="0 0 -1.0472" xyz="0.018 0 0"/>
-		<axis xyz="0 0 1.0"/>
-		<mimic joint="RHand" multiplier="0.872665" offset="0"/>
-	</joint>
-	<link name="LFinger22_link">
-		<xacro:insert_visu_LFinger22_link/>
-	</link>
-	<joint name="LFinger22" type="continuous">
-		<parent link="LFinger21_link"/>
-		<child link="LFinger22_link"/>
-		<origin rpy="0 0 -1.0472" xyz="0.018 0 0"/>
-		<axis xyz="0 0 1.0"/>
-		<mimic joint="LHand" multiplier="0.872665" offset="0"/>
-	</joint>
-	<link name="RFinger21_link">
-		<xacro:insert_visu_RFinger21_link/>
-	</link>
-	<joint name="RFinger21" type="continuous">
-		<parent link="r_wrist"/>
-		<child link="RFinger21_link"/>
-		<origin rpy="1.5708 1.0472 0.061086" xyz="0.0873 0.0073 0.006"/>
-		<axis xyz="0 0 1.0"/>
-		<mimic joint="RHand" multiplier="0.872665" offset="0"/>
-	</joint>
-	<link name="LFinger12_link">
-		<xacro:insert_visu_LFinger12_link/>
-	</link>
-	<joint name="LFinger12" type="continuous">
-		<parent link="LFinger11_link"/>
-		<child link="LFinger12_link"/>
-		<origin rpy="0 0 -1.0472" xyz="0.018 0 0"/>
-		<axis xyz="0 0 1.0"/>
-		<mimic joint="LHand" multiplier="0.872665" offset="0"/>
-	</joint>
-	<link name="RFinger23_link">
-		<xacro:insert_visu_RFinger23_link/>
-	</link>
-	<joint name="RFinger23" type="continuous">
-		<parent link="RFinger22_link"/>
-		<child link="RFinger23_link"/>
-		<origin rpy="0 0 -1.0472" xyz="0.018 0 0"/>
-		<axis xyz="0 0 1.0"/>
-		<mimic joint="RHand" multiplier="0.872665" offset="0"/>
-	</joint>
-	<link name="LFinger23_link">
-		<xacro:insert_visu_LFinger23_link/>
-	</link>
-	<joint name="LFinger23" type="continuous">
-		<parent link="LFinger22_link"/>
-		<child link="LFinger23_link"/>
-		<origin rpy="0 0 -1.0472" xyz="0.018 0 0"/>
-		<axis xyz="0 0 1.0"/>
-		<mimic joint="LHand" multiplier="0.872665" offset="0"/>
-	</joint>
-	<link name="LFinger43_link">
-		<xacro:insert_visu_LFinger43_link/>
-	</link>
-	<joint name="LFinger43" type="continuous">
-		<parent link="LFinger42_link"/>
-		<child link="LFinger43_link"/>
-		<origin rpy="0 0 -1.0472" xyz="0.018 0 0"/>
-		<axis xyz="0 0 1.0"/>
-		<mimic joint="LHand" multiplier="0.872665" offset="0"/>
-	</joint>
 	<link name="RFinger42_link">
+		<inertial>
+			<mass value="2e-06"/>
+			<inertia ixx="1.1e-09" ixy="0" ixz="0" iyy="1.1e-09" iyz="0" izz="1.1e-09"/>
+		</inertial>
 		<xacro:insert_visu_RFinger42_link/>
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
File: pepper_description/urdf/pepper1.0_generated_urdf/pepper_robot.xacro (robot description, xacro)
@@ -3,5 +3,5 @@
  ****** File automatically generated by generate_urdf.py script ******
  *********************************************************************-->
-<robot name="julietteY20MP" xmlns:xacro="http://www.ros.org/wiki/xacro">
+<robot name="JulietteY20MP" xmlns:xacro="http://www.ros.org/wiki/xacro">
 	<xacro:include filename="pepper_visual_collisions.xacro"/>
 	<xacro:include filename="pepper_head.xacro"/>

File: pepper_description/urdf/pepper1.0_generated_urdf/pepper_sensors.xacro (robot description, xacro)
@@ -3,5 +3,5 @@
  ****** File automatically generated by generate_urdf.py script ******
  *********************************************************************-->
-<robot name="julietteY20MP" xmlns:xacro="http://www.ros.org/wiki/xacro">
+<robot name="JulietteY20MP" xmlns:xacro="http://www.ros.org/wiki/xacro">
 	<link name="SonarBack_frame"/>
 	<joint name="Sonar/Back_sensor_fixedjoint" type="fixed">
@@ -12,5 +12,5 @@
 	</joint>
 	<link name="CameraBottom_optical_frame"/>
-	<joint name="CameraBottom_optical_frame_joint" type="fixed">
+	<joint name="CameraBottom_optical_frame_fixedjoint" type="fixed">
 		<parent link="CameraBottom_frame"/>
 		<child link="CameraBottom_optical_frame"/>
@@ -18,5 +18,5 @@
 	</joint>
 	<link name="CameraDepth_optical_frame"/>
-	<joint name="CameraDepth_optical_frame_joint" type="fixed">
+	<joint name="CameraDepth_optical_frame_fixedjoint" type="fixed">
 		<parent link="CameraDepth_frame"/>
 		<child link="CameraDepth_optical_frame"/>
@@ -30,11 +30,4 @@
 		<axis xyz="0 0 0"/>
 	</joint>
-	<link name="SurroundingFrontLaser_frame"/>
-	<joint name="LaserSensor/Front_sensor_fixedjoint" type="fixed">
-		<parent link="Tibia"/>
-		<child link="SurroundingFrontLaser_frame"/>
-		<origin rpy="0 0 0" xyz="0.0562 0 -0.334"/>
-		<axis xyz="0 0 0"/>
-	</joint>
 	<link name="VerticalLeftLaser_frame"/>
 	<joint name="LaserSensor/VerticalLeft_sensor_fixedjoint" type="fixed">
@@ -44,4 +37,11 @@
 		<axis xyz="0 0 0"/>
 	</joint>
+	<link name="SurroundingFrontLaser_device_frame"/>
+	<joint name="LaserSensor/Front_sensor_fixedjoint" type="fixed">
+		<parent link="Tibia"/>
+		<child link="SurroundingFrontLaser_device_frame"/>
+		<origin rpy="0 0.349044 0" xyz="0.0562 0 -0.0692"/>
+		<axis xyz="0 0 0"/>
+	</joint>
 	<link name="BumperB_frame"/>
 	<joint name="Bumper/Back_sensor_fixedjoint" type="fixed">
@@ -52,8 +52,8 @@
 	</joint>
 	<link name="SurroundingLeftLaser_frame"/>
-	<joint name="LaserSensor/Left_sensor_fixedjoint" type="fixed">
+	<joint name="LaserSensor/Left_projected_sensor_fixedjoint" type="fixed">
 		<parent link="Tibia"/>
 		<child link="SurroundingLeftLaser_frame"/>
-		<origin rpy="0 0 ${1.5708+0.1864836732051034}" xyz="-0.018 0.0899 -0.334"/>
+		<origin rpy="0 0 1.75728" xyz="-0.018 0.0899 -0.334"/>
 		<axis xyz="0 0 0"/>
 	</joint>
@@ -72,9 +72,16 @@
 		<axis xyz="0 0 0"/>
 	</joint>
-	<link name="ImuTorsoGyrometer_frame"/>
-	<joint name="Gyrometer_sensor_fixedjoint" type="fixed">
-		<parent link="torso"/>
-		<child link="ImuTorsoGyrometer_frame"/>
-		<origin rpy="0 0 0" xyz="0.00204 -0.03491 -0.00959"/>
+	<link name="CameraTop_frame"/>
+	<joint name="CameraTop_sensor_fixedjoint" type="fixed">
+		<parent link="Head"/>
+		<child link="CameraTop_frame"/>
+		<origin rpy="0 0 0" xyz="0.0868 0 0.1631"/>
+		<axis xyz="0 0 0"/>
+	</joint>
+	<link name="SurroundingRightLaser_device_frame"/>
+	<joint name="LaserSensor/Right_sensor_fixedjoint" type="fixed">
+		<parent link="Tibia"/>
+		<child link="SurroundingRightLaser_device_frame"/>
+		<origin rpy="4.08851e-07 0.191857 -1.60746" xyz="-0.018 -0.0899 -0.0759"/>
 		<axis xyz="0 0 0"/>
 	</joint>
@@ -100,4 +107,11 @@
 		<axis xyz="0 0 0"/>
 	</joint>
+	<link name="SurroundingLeftLaser_device_frame"/>
+	<joint name="LaserSensor/Left_sensor_fixedjoint" type="fixed">
+		<parent link="Tibia"/>
+		<child link="SurroundingLeftLaser_device_frame"/>
+		<origin rpy="8.34035e-09 0.191982 1.5708" xyz="-0.018 0.0899 -0.0759"/>
+		<axis xyz="0 0 0"/>
+	</joint>
 	<link name="CameraDepth_frame"/>
 	<joint name="CameraDepth_sensor_fixedjoint" type="fixed">
@@ -108,8 +122,8 @@
 	</joint>
 	<link name="SurroundingRightLaser_frame"/>
-	<joint name="LaserSensor/Right_sensor_fixedjoint" type="fixed">
+	<joint name="LaserSensor/Right_projected_sensor_fixedjoint" type="fixed">
 		<parent link="Tibia"/>
 		<child link="SurroundingRightLaser_frame"/>
-		<origin rpy="0 0 ${-1.5708-0.1864836732051034}" xyz="-0.018 -0.0899 -0.334"/>
+		<origin rpy="0 0 -1.75728" xyz="-0.018 -0.0899 -0.334"/>
 		<axis xyz="0 0 0"/>
 	</joint>
@@ -135,4 +149,11 @@
 		<axis xyz="0 0 0"/>
 	</joint>
+	<link name="BumperFL_frame"/>
+	<joint name="Bumper/FrontLeft_sensor_fixedjoint" type="fixed">
+		<parent link="Tibia"/>
+		<child link="BumperFL_frame"/>
+		<origin rpy="0 0 0.48886" xyz="0.129 0.227 -0.264"/>
+		<axis xyz="0 0 0"/>
+	</joint>
 	<link name="CameraBottom_frame"/>
 	<joint name="CameraBottom_sensor_fixedjoint" type="fixed">
@@ -142,13 +163,6 @@
 		<axis xyz="0 0 0"/>
 	</joint>
-	<link name="CameraTop_frame"/>
-	<joint name="CameraTop_sensor_fixedjoint" type="fixed">
-		<parent link="Head"/>
-		<child link="CameraTop_frame"/>
-		<origin rpy="0 0 0" xyz="0.0868 0 0.1631"/>
-		<axis xyz="0 0 0"/>
-	</joint>
 	<link name="CameraTop_optical_frame"/>
-	<joint name="CameraTop_optical_frame_joint" type="fixed">
+	<joint name="CameraTop_optical_frame_fixedjoint" type="fixed">
 		<parent link="CameraTop_frame"/>
 		<child link="CameraTop_optical_frame"/>
@@ -162,9 +176,9 @@
 		<axis xyz="0 0 0"/>
 	</joint>
-	<link name="BumperFL_frame"/>
-	<joint name="Bumper/FrontLeft_sensor_fixedjoint" type="fixed">
-		<parent link="Tibia"/>
-		<child link="BumperFL_frame"/>
-		<origin rpy="0 0 0.48886" xyz="0.129 0.227 -0.264"/>
+	<link name="ImuTorsoGyrometer_frame"/>
+	<joint name="Gyrometer_sensor_fixedjoint" type="fixed">
+		<parent link="torso"/>
+		<child link="ImuTorsoGyrometer_frame"/>
+		<origin rpy="0 0 0" xyz="0.00204 -0.03491 -0.00959"/>
 		<axis xyz="0 0 0"/>
 	</joint>
@@ -190,4 +204,11 @@
 		<axis xyz="0 0 0"/>
 	</joint>
+	<link name="SurroundingFrontLaser_frame"/>
+	<joint name="LaserSensor/Front_projected_sensor_fixedjoint" type="fixed">
+		<parent link="Tibia"/>
+		<child link="SurroundingFrontLaser_frame"/>
+		<origin rpy="0 0 0" xyz="0.0562 0 -0.334"/>
+		<axis xyz="0 0 0"/>
+	</joint>
 	<link name="ChestButton_frame"/>
 	<joint name="ChestBoard/Button_sensor_fixedjoint" type="fixed">
