Commit message: update to the latest alrobotmodelutils

File: pepper_description/urdf/pepper1.0_generated_urdf/pepper_visual_collisions.xacro (robot description, xacro)
@@ -102,4 +102,508 @@
 		</collision>
 	</xacro:macro>
+	<xacro:macro name="xacro:insert_visu_RFinger31_link">
+		<visual>
+			<geometry>
+				<mesh filename="package://pepper_meshes/meshes/1.0/RFinger31.dae" scale="0.1 0.1 0.1"/>
+			</geometry>
+			<origin rpy="0 0 0" xyz="0 0 0"/>
+		</visual>
+		<collision>
+			<geometry>
+				<mesh filename="package://pepper_meshes/meshes/1.0/RFinger31_0.10.stl" scale="0.1 0.1 0.1"/>
+			</geometry>
+			<origin rpy="0 0 0" xyz="0 0 0"/>
+		</collision>
+	</xacro:macro>
+	<xacro:macro name="xacro:insert_visu_LFinger21_link">
+		<visual>
+			<geometry>
+				<mesh filename="package://pepper_meshes/meshes/1.0/LFinger21.dae" scale="0.1 0.1 0.1"/>
+			</geometry>
+			<origin rpy="0 0 0" xyz="0 0 0"/>
+		</visual>
+		<collision>
+			<geometry>
+				<mesh filename="package://pepper_meshes/meshes/1.0/LFinger21_0.10.stl" scale="0.1 0.1 0.1"/>
+			</geometry>
+			<origin rpy="0 0 0" xyz="0 0 0"/>
+		</collision>
+	</xacro:macro>
+	<xacro:macro name="xacro:insert_visu_RFinger32_link">
+		<visual>
+			<geometry>
+				<mesh filename="package://pepper_meshes/meshes/1.0/RFinger32.dae" scale="0.1 0.1 0.1"/>
+			</geometry>
+			<origin rpy="0 0 0" xyz="0 0 0"/>
+		</visual>
+		<collision>
+			<geometry>
+				<mesh filename="package://pepper_meshes/meshes/1.0/RFinger32_0.10.stl" scale="0.1 0.1 0.1"/>
+			</geometry>
+			<origin rpy="0 0 0" xyz="0 0 0"/>
+		</collision>
+	</xacro:macro>
+	<xacro:macro name="xacro:insert_visu_LFinger13_link">
+		<visual>
+			<geometry>
+				<mesh filename="package://pepper_meshes/meshes/1.0/LFinger13.dae" scale="0.1 0.1 0.1"/>
+			</geometry>
+			<origin rpy="0 0 0" xyz="0 0 0"/>
+		</visual>
+		<collision>
+			<geometry>
+				<mesh filename="package://pepper_meshes/meshes/1.0/LFinger13_0.10.stl" scale="0.1 0.1 0.1"/>
+			</geometry>
+			<origin rpy="0 0 0" xyz="0 0 0"/>
+		</collision>
+	</xacro:macro>
+	<xacro:macro name="xacro:insert_visu_LFinger32_link">
+		<visual>
+			<geometry>
+				<mesh filename="package://pepper_meshes/meshes/1.0/LFinger32.dae" scale="0.1 0.1 0.1"/>
+			</geometry>
+			<origin rpy="0 0 0" xyz="0 0 0"/>
+		</visual>
+		<collision>
+			<geometry>
+				<mesh filename="package://pepper_meshes/meshes/1.0/LFinger32_0.10.stl" scale="0.1 0.1 0.1"/>
+			</geometry>
+			<origin rpy="0 0 0" xyz="0 0 0"/>
+		</collision>
+	</xacro:macro>
+	<xacro:macro name="xacro:insert_visu_LThumb1_link">
+		<visual>
+			<geometry>
+				<mesh filename="package://pepper_meshes/meshes/1.0/LThumb1.dae" scale="0.1 0.1 0.1"/>
+			</geometry>
+			<origin rpy="0 0 0" xyz="0 0 0"/>
+		</visual>
+		<collision>
+			<geometry>
+				<mesh filename="package://pepper_meshes/meshes/1.0/LThumb1_0.10.stl" scale="0.1 0.1 0.1"/>
+			</geometry>
+			<origin rpy="0 0 0" xyz="0 0 0"/>
+		</collision>
+	</xacro:macro>
+	<xacro:macro name="xacro:insert_visu_LFinger11_link">
+		<visual>
+			<geometry>
+				<mesh filename="package://pepper_meshes/meshes/1.0/LFinger11.dae" scale="0.1 0.1 0.1"/>
+			</geometry>
+			<origin rpy="0 0 0" xyz="0 0 0"/>
+		</visual>
+		<collision>
+			<geometry>
+				<mesh filename="package://pepper_meshes/meshes/1.0/LFinger11_0.10.stl" scale="0.1 0.1 0.1"/>
+			</geometry>
+			<origin rpy="0 0 0" xyz="0 0 0"/>
+		</collision>
+	</xacro:macro>
+	<xacro:macro name="xacro:insert_visu_RFinger22_link">
+		<visual>
+			<geometry>
+				<mesh filename="package://pepper_meshes/meshes/1.0/RFinger22.dae" scale="0.1 0.1 0.1"/>
+			</geometry>
+			<origin rpy="0 0 0" xyz="0 0 0"/>
+		</visual>
+		<collision>
+			<geometry>
+				<mesh filename="package://pepper_meshes/meshes/1.0/RFinger22_0.10.stl" scale="0.1 0.1 0.1"/>
+			</geometry>
+			<origin rpy="0 0 0" xyz="0 0 0"/>
+		</collision>
+	</xacro:macro>
+	<xacro:macro name="xacro:insert_visu_RThumb2_link">
+		<visual>
+			<geometry>
+				<mesh filename="package://pepper_meshes/meshes/1.0/RThumb2.dae" scale="0.1 0.1 0.1"/>
+			</geometry>
+			<origin rpy="0 0 0" xyz="0 0 0"/>
+		</visual>
+		<collision>
+			<geometry>
+				<mesh filename="package://pepper_meshes/meshes/1.0/RThumb2_0.10.stl" scale="0.1 0.1 0.1"/>
+			</geometry>
+			<origin rpy="0 0 0" xyz="0 0 0"/>
+		</collision>
+	</xacro:macro>
+	<xacro:macro name="xacro:insert_visu_RFinger13_link">
+		<visual>
+			<geometry>
+				<mesh filename="package://pepper_meshes/meshes/1.0/RFinger13.dae" scale="0.1 0.1 0.1"/>
+			</geometry>
+			<origin rpy="0 0 0" xyz="0 0 0"/>
+		</visual>
+		<collision>
+			<geometry>
+				<mesh filename="package://pepper_meshes/meshes/1.0/RFinger13_0.10.stl" scale="0.1 0.1 0.1"/>
+			</geometry>
+			<origin rpy="0 0 0" xyz="0 0 0"/>
+		</collision>
+	</xacro:macro>
+	<xacro:macro name="xacro:insert_visu_Tibia">
+		<visual>
+			<geometry>
+				<mesh filename="package://pepper_meshes/meshes/1.0/KneePitch.dae" scale="0.1 0.1 0.1"/>
+			</geometry>
+			<origin rpy="0 0 0" xyz="0 0 0"/>
+		</visual>
+		<collision>
+			<geometry>
+				<mesh filename="package://pepper_meshes/meshes/1.0/KneePitch_0.10.stl" scale="0.1 0.1 0.1"/>
+			</geometry>
+			<origin rpy="0 0 0" xyz="0 0 0"/>
+		</collision>
+	</xacro:macro>
+	<xacro:macro name="xacro:insert_visu_Head">
+		<visual>
+			<geometry>
+				<mesh filename="package://pepper_meshes/meshes/1.0/HeadPitch.dae" scale="0.1 0.1 0.1"/>
+			</geometry>
+			<origin rpy="0 0 0" xyz="0 0 0"/>
+		</visual>
+		<collision>
+			<geometry>
+				<mesh filename="package://pepper_meshes/meshes/1.0/HeadPitch_0.10.stl" scale="0.1 0.1 0.1"/>
+			</geometry>
+			<origin rpy="0 0 0" xyz="0 0 0"/>
+		</collision>
+	</xacro:macro>
+	<xacro:macro name="xacro:insert_visu_LFinger22_link">
+		<visual>
+			<geometry>
+				<mesh filename="package://pepper_meshes/meshes/1.0/LFinger22.dae" scale="0.1 0.1 0.1"/>
+			</geometry>
+			<origin rpy="0 0 0" xyz="0 0 0"/>
+		</visual>
+		<collision>
+			<geometry>
+				<mesh filename="package://pepper_meshes/meshes/1.0/LFinger22_0.10.stl" scale="0.1 0.1 0.1"/>
+			</geometry>
+			<origin rpy="0 0 0" xyz="0 0 0"/>
+		</collision>
+	</xacro:macro>
+	<xacro:macro name="xacro:insert_visu_RFinger21_link">
+		<visual>
+			<geometry>
+				<mesh filename="package://pepper_meshes/meshes/1.0/RFinger21.dae" scale="0.1 0.1 0.1"/>
+			</geometry>
+			<origin rpy="0 0 0" xyz="0 0 0"/>
+		</visual>
+		<collision>
+			<geometry>
+				<mesh filename="package://pepper_meshes/meshes/1.0/RFinger21_0.10.stl" scale="0.1 0.1 0.1"/>
+			</geometry>
+			<origin rpy="0 0 0" xyz="0 0 0"/>
+		</collision>
+	</xacro:macro>
+	<xacro:macro name="xacro:insert_visu_LBicep">
+		<visual>
+			<geometry>
+				<mesh filename="package://pepper_meshes/meshes/1.0/LShoulderRoll.dae" scale="0.1 0.1 0.1"/>
+			</geometry>
+			<origin rpy="0 0 0" xyz="0 0 0"/>
+		</visual>
+		<collision>
+			<geometry>
+				<mesh filename="package://pepper_meshes/meshes/1.0/LShoulderRoll_0.10.stl" scale="0.1 0.1 0.1"/>
+			</geometry>
+			<origin rpy="0 0 0" xyz="0 0 0"/>
+		</collision>
+	</xacro:macro>
+	<xacro:macro name="xacro:insert_visu_RThumb1_link">
+		<visual>
+			<geometry>
+				<mesh filename="package://pepper_meshes/meshes/1.0/RThumb1.dae" scale="0.1 0.1 0.1"/>
+			</geometry>
+			<origin rpy="0 0 0" xyz="0 0 0"/>
+		</visual>
+		<collision>
+			<geometry>
+				<mesh filename="package://pepper_meshes/meshes/1.0/RThumb1_0.10.stl" scale="0.1 0.1 0.1"/>
+			</geometry>
+			<origin rpy="0 0 0" xyz="0 0 0"/>
+		</collision>
+	</xacro:macro>
+	<xacro:macro name="xacro:insert_visu_LFinger41_link">
+		<visual>
+			<geometry>
+				<mesh filename="package://pepper_meshes/meshes/1.0/LFinger41.dae" scale="0.1 0.1 0.1"/>
+			</geometry>
+			<origin rpy="0 0 0" xyz="0 0 0"/>
+		</visual>
+		<collision>
+			<geometry>
+				<mesh filename="package://pepper_meshes/meshes/1.0/LFinger41_0.10.stl" scale="0.1 0.1 0.1"/>
+			</geometry>
+			<origin rpy="0 0 0" xyz="0 0 0"/>
+		</collision>
+	</xacro:macro>
+	<xacro:macro name="xacro:insert_visu_r_wrist">
+		<visual>
+			<geometry>
+				<mesh filename="package://pepper_meshes/meshes/1.0/RWristYaw.dae" scale="0.1 0.1 0.1"/>
+			</geometry>
+			<origin rpy="0 0 0" xyz="0 0 0"/>
+		</visual>
+		<collision>
+			<geometry>
+				<mesh filename="package://pepper_meshes/meshes/1.0/RWristYaw_0.10.stl" scale="0.1 0.1 0.1"/>
+			</geometry>
+			<origin rpy="0 0 0" xyz="0 0 0"/>
+		</collision>
+	</xacro:macro>
+	<xacro:macro name="xacro:insert_visu_LForeArm">
+		<visual>
+			<geometry>
+				<mesh filename="package://pepper_meshes/meshes/1.0/LElbowRoll.dae" scale="0.1 0.1 0.1"/>
+			</geometry>
+			<origin rpy="0 0 0" xyz="0 0 0"/>
+		</visual>
+		<collision>
+			<geometry>
+				<mesh filename="package://pepper_meshes/meshes/1.0/LElbowRoll_0.10.stl" scale="0.1 0.1 0.1"/>
+			</geometry>
+			<origin rpy="0 0 0" xyz="0 0 0"/>
+		</collision>
+	</xacro:macro>
+	<xacro:macro name="xacro:insert_visu_LThumb2_link">
+		<visual>
+			<geometry>
+				<mesh filename="package://pepper_meshes/meshes/1.0/LThumb2.dae" scale="0.1 0.1 0.1"/>
+			</geometry>
+			<origin rpy="0 0 0" xyz="0 0 0"/>
+		</visual>
+		<collision>
+			<geometry>
+				<mesh filename="package://pepper_meshes/meshes/1.0/LThumb2_0.10.stl" scale="0.1 0.1 0.1"/>
+			</geometry>
+			<origin rpy="0 0 0" xyz="0 0 0"/>
+		</collision>
+	</xacro:macro>
+	<xacro:macro name="xacro:insert_visu_LFinger12_link">
+		<visual>
+			<geometry>
+				<mesh filename="package://pepper_meshes/meshes/1.0/LFinger12.dae" scale="0.1 0.1 0.1"/>
+			</geometry>
+			<origin rpy="0 0 0" xyz="0 0 0"/>
+		</visual>
+		<collision>
+			<geometry>
+				<mesh filename="package://pepper_meshes/meshes/1.0/LFinger12_0.10.stl" scale="0.1 0.1 0.1"/>
+			</geometry>
+			<origin rpy="0 0 0" xyz="0 0 0"/>
+		</collision>
+	</xacro:macro>
+	<xacro:macro name="xacro:insert_visu_RShoulder">
+		<visual>
+			<geometry>
+				<mesh filename="package://pepper_meshes/meshes/1.0/RShoulderPitch.dae" scale="0.1 0.1 0.1"/>
+			</geometry>
+			<origin rpy="0 0 0" xyz="0 0 0"/>
+		</visual>
+		<collision>
+			<geometry>
+				<mesh filename="package://pepper_meshes/meshes/1.0/RShoulderPitch_0.10.stl" scale="0.1 0.1 0.1"/>
+			</geometry>
+			<origin rpy="0 0 0" xyz="0 0 0"/>
+		</collision>
+	</xacro:macro>
+	<xacro:macro name="xacro:insert_visu_RFinger23_link">
+		<visual>
+			<geometry>
+				<mesh filename="package://pepper_meshes/meshes/1.0/RFinger23.dae" scale="0.1 0.1 0.1"/>
+			</geometry>
+			<origin rpy="0 0 0" xyz="0 0 0"/>
+		</visual>
+		<collision>
+			<geometry>
+				<mesh filename="package://pepper_meshes/meshes/1.0/RFinger23_0.10.stl" scale="0.1 0.1 0.1"/>
+			</geometry>
+			<origin rpy="0 0 0" xyz="0 0 0"/>
+		</collision>
+	</xacro:macro>
+	<xacro:macro name="xacro:insert_visu_l_wrist">
+		<visual>
+			<geometry>
+				<mesh filename="package://pepper_meshes/meshes/1.0/LWristYaw.dae" scale="0.1 0.1 0.1"/>
+			</geometry>
+			<origin rpy="0 0 0" xyz="0 0 0"/>
+		</visual>
+		<collision>
+			<geometry>
+				<mesh filename="package://pepper_meshes/meshes/1.0/LWristYaw_0.10.stl" scale="0.1 0.1 0.1"/>
+			</geometry>
+			<origin rpy="0 0 0" xyz="0 0 0"/>
+		</collision>
+	</xacro:macro>
+	<xacro:macro name="xacro:insert_visu_RBicep">
+		<visual>
+			<geometry>
+				<mesh filename="package://pepper_meshes/meshes/1.0/RShoulderRoll.dae" scale="0.1 0.1 0.1"/>
+			</geometry>
+			<origin rpy="0 0 0" xyz="0 0 0"/>
+		</visual>
+		<collision>
+			<geometry>
+				<mesh filename="package://pepper_meshes/meshes/1.0/RShoulderRoll_0.10.stl" scale="0.1 0.1 0.1"/>
+			</geometry>
+			<origin rpy="0 0 0" xyz="0 0 0"/>
+		</collision>
+	</xacro:macro>
+	<xacro:macro name="xacro:insert_visu_WheelB_link">
+		<visual>
+			<geometry>
+				<mesh filename="package://pepper_meshes/meshes/1.0/WheelB.dae" scale="0.1 0.1 0.1"/>
+			</geometry>
+			<origin rpy="0 0 0" xyz="0 0 0"/>
+		</visual>
+		<collision>
+			<geometry>
+				<mesh filename="package://pepper_meshes/meshes/1.0/WheelB_0.10.stl" scale="0.1 0.1 0.1"/>
+			</geometry>
+			<origin rpy="0 0 0" xyz="0 0 0"/>
+		</collision>
+	</xacro:macro>
+	<xacro:macro name="xacro:insert_visu_LFinger23_link">
+		<visual>
+			<geometry>
+				<mesh filename="package://pepper_meshes/meshes/1.0/LFinger23.dae" scale="0.1 0.1 0.1"/>
+			</geometry>
+			<origin rpy="0 0 0" xyz="0 0 0"/>
+		</visual>
+		<collision>
+			<geometry>
+				<mesh filename="package://pepper_meshes/meshes/1.0/LFinger23_0.10.stl" scale="0.1 0.1 0.1"/>
+			</geometry>
+			<origin rpy="0 0 0" xyz="0 0 0"/>
+		</collision>
+	</xacro:macro>
+	<xacro:macro name="xacro:insert_visu_RElbow">
+		<visual>
+			<geometry>
+				<mesh filename="package://pepper_meshes/meshes/1.0/RElbowYaw.dae" scale="0.1 0.1 0.1"/>
+			</geometry>
+			<origin rpy="0 0 0" xyz="0 0 0"/>
+		</visual>
+		<collision>
+			<geometry>
+				<mesh filename="package://pepper_meshes/meshes/1.0/RElbowYaw_0.10.stl" scale="0.1 0.1 0.1"/>
+			</geometry>
+			<origin rpy="0 0 0" xyz="0 0 0"/>
+		</collision>
+	</xacro:macro>
+	<xacro:macro name="xacro:insert_visu_Neck">
+		<visual>
+			<geometry>
+				<mesh filename="package://pepper_meshes/meshes/1.0/HeadYaw.dae" scale="0.1 0.1 0.1"/>
+			</geometry>
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
File: pepper_description/urdf/pepper1.0_generated_urdf/pepper_wheels.xacro (robot description, xacro)
@@ -3,5 +3,20 @@
  ****** File automatically generated by generate_urdf.py script ******
  *********************************************************************-->
-<robot name="julietteY20MP" xmlns:xacro="http://www.ros.org/wiki/xacro">
+<robot name="JulietteY20MP" xmlns:xacro="http://www.ros.org/wiki/xacro">
+	<link name="WheelB_link">
+		<inertial>
+			<mass value="1.58028"/>
+			<inertia ixx="0.00299756" ixy="-6.3068e-07" ixz="-5.56903e-06" iyy="0.00303229" iyz="9.0408e-07" izz="0.00296585"/>
+			<origin rpy="0 0 0" xyz="0 0 0"/>
+		</inertial>
+		<xacro:insert_visu_WheelB_link/>
+	</link>
+	<joint name="WheelB" type="continuous">
+		<parent link="Tibia"/>
+		<child link="WheelB_link"/>
+		<origin rpy="0 0 -3.14159" xyz="-0.17 0 -0.264"/>
+		<axis xyz="1.0 0 0"/>
+		<limit effort="3.25" lower="0" upper="0" velocity="6.28319"/>
+	</joint>
 	<link name="WheelFL_link">
 		<inertial>
@@ -16,19 +31,4 @@
 		<child link="WheelFL_link"/>
 		<origin rpy="0 0 1.07517" xyz="0.09 0.155 -0.264"/>
-		<axis xyz="1.0 0 0"/>
-		<limit effort="3.25" lower="0" upper="0" velocity="6.28319"/>
-	</joint>
-	<link name="WheelB_link">
-		<inertial>
-			<mass value="1.58028"/>
-			<inertia ixx="0.00299756" ixy="-6.3068e-07" ixz="-5.56903e-06" iyy="0.00303229" iyz="9.0408e-07" izz="0.00296585"/>
-			<origin rpy="0 0 0" xyz="0 0 0"/>
-		</inertial>
-		<xacro:insert_visu_WheelB_link/>
-	</link>
-	<joint name="WheelB" type="continuous">
-		<parent link="Tibia"/>
-		<child link="WheelB_link"/>
-		<origin rpy="0 0 -3.14159" xyz="-0.17 0 -0.264"/>
 		<axis xyz="1.0 0 0"/>
 		<limit effort="3.25" lower="0" upper="0" velocity="6.28319"/>
