Commit message: use proper macro names

File: pepper_description/urdf/pepper1.0_generated_urdf/pepper_visual_collisions.xacro (robot description, xacro)
@@ -4,5 +4,5 @@
  *********************************************************************-->
 <robot xmlns:xacro="http://www.ros.org/wiki/xacro">
-	<xacro:macro name="xacro:insert_visu_RFinger41_link">
+	<xacro:macro name="insert_visu_RFinger41_link">
 		<visual>
 			<geometry>
@@ -18,5 +18,5 @@
 		</collision>
 	</xacro:macro>
-	<xacro:macro name="xacro:insert_visu_LFinger42_link">
+	<xacro:macro name="insert_visu_LFinger42_link">
 		<visual>
 			<geometry>
@@ -32,5 +32,5 @@
 		</collision>
 	</xacro:macro>
-	<xacro:macro name="xacro:insert_visu_Hip">
+	<xacro:macro name="insert_visu_Hip">
 		<visual>
 			<geometry>
@@ -46,5 +46,5 @@
 		</collision>
 	</xacro:macro>
-	<xacro:macro name="xacro:insert_visu_RFinger11_link">
+	<xacro:macro name="insert_visu_RFinger11_link">
 		<visual>
 			<geometry>
@@ -60,5 +60,5 @@
 		</collision>
 	</xacro:macro>
-	<xacro:macro name="xacro:insert_visu_LElbow">
+	<xacro:macro name="insert_visu_LElbow">
 		<visual>
 			<geometry>
@@ -74,5 +74,5 @@
 		</collision>
 	</xacro:macro>
-	<xacro:macro name="xacro:insert_visu_RFinger12_link">
+	<xacro:macro name="insert_visu_RFinger12_link">
 		<visual>
 			<geometry>
@@ -88,5 +88,5 @@
 		</collision>
 	</xacro:macro>
-	<xacro:macro name="xacro:insert_visu_LFinger33_link">
+	<xacro:macro name="insert_visu_LFinger33_link">
 		<visual>
 			<geometry>
@@ -102,5 +102,5 @@
 		</collision>
 	</xacro:macro>
-	<xacro:macro name="xacro:insert_visu_RFinger31_link">
+	<xacro:macro name="insert_visu_RFinger31_link">
 		<visual>
 			<geometry>
@@ -116,5 +116,5 @@
 		</collision>
 	</xacro:macro>
-	<xacro:macro name="xacro:insert_visu_LFinger21_link">
+	<xacro:macro name="insert_visu_LFinger21_link">
 		<visual>
 			<geometry>
@@ -130,5 +130,5 @@
 		</collision>
 	</xacro:macro>
-	<xacro:macro name="xacro:insert_visu_RFinger32_link">
+	<xacro:macro name="insert_visu_RFinger32_link">
 		<visual>
 			<geometry>
@@ -144,5 +144,5 @@
 		</collision>
 	</xacro:macro>
-	<xacro:macro name="xacro:insert_visu_LFinger13_link">
+	<xacro:macro name="insert_visu_LFinger13_link">
 		<visual>
 			<geometry>
@@ -158,5 +158,5 @@
 		</collision>
 	</xacro:macro>
-	<xacro:macro name="xacro:insert_visu_LFinger32_link">
+	<xacro:macro name="insert_visu_LFinger32_link">
 		<visual>
 			<geometry>
@@ -172,5 +172,5 @@
 		</collision>
 	</xacro:macro>
-	<xacro:macro name="xacro:insert_visu_LThumb1_link">
+	<xacro:macro name="insert_visu_LThumb1_link">
 		<visual>
 			<geometry>
@@ -186,5 +186,5 @@
 		</collision>
 	</xacro:macro>
-	<xacro:macro name="xacro:insert_visu_LFinger11_link">
+	<xacro:macro name="insert_visu_LFinger11_link">
 		<visual>
 			<geometry>
@@ -200,5 +200,5 @@
 		</collision>
 	</xacro:macro>
-	<xacro:macro name="xacro:insert_visu_RFinger22_link">
+	<xacro:macro name="insert_visu_RFinger22_link">
 		<visual>
 			<geometry>
@@ -214,5 +214,5 @@
 		</collision>
 	</xacro:macro>
-	<xacro:macro name="xacro:insert_visu_RThumb2_link">
+	<xacro:macro name="insert_visu_RThumb2_link">
 		<visual>
 			<geometry>
@@ -228,5 +228,5 @@
 		</collision>
 	</xacro:macro>
-	<xacro:macro name="xacro:insert_visu_RFinger13_link">
+	<xacro:macro name="insert_visu_RFinger13_link">
 		<visual>
 			<geometry>
@@ -242,5 +242,5 @@
 		</collision>
 	</xacro:macro>
-	<xacro:macro name="xacro:insert_visu_Tibia">
+	<xacro:macro name="insert_visu_Tibia">
 		<visual>
 			<geometry>
@@ -256,5 +256,5 @@
 		</collision>
 	</xacro:macro>
-	<xacro:macro name="xacro:insert_visu_Head">
+	<xacro:macro name="insert_visu_Head">
 		<visual>
 			<geometry>
@@ -270,5 +270,5 @@
 		</collision>
 	</xacro:macro>
-	<xacro:macro name="xacro:insert_visu_LFinger22_link">
+	<xacro:macro name="insert_visu_LFinger22_link">
 		<visual>
 			<geometry>
@@ -284,5 +284,5 @@
 		</collision>
 	</xacro:macro>
-	<xacro:macro name="xacro:insert_visu_RFinger21_link">
+	<xacro:macro name="insert_visu_RFinger21_link">
 		<visual>
 			<geometry>
@@ -298,5 +298,5 @@
 		</collision>
 	</xacro:macro>
-	<xacro:macro name="xacro:insert_visu_LBicep">
+	<xacro:macro name="insert_visu_LBicep">
 		<visual>
 			<geometry>
@@ -312,5 +312,5 @@
 		</collision>
 	</xacro:macro>
-	<xacro:macro name="xacro:insert_visu_RThumb1_link">
+	<xacro:macro name="insert_visu_RThumb1_link">
 		<visual>
 			<geometry>
@@ -326,5 +326,5 @@
 		</collision>
 	</xacro:macro>
-	<xacro:macro name="xacro:insert_visu_LFinger41_link">
+	<xacro:macro name="insert_visu_LFinger41_link">
 		<visual>
 			<geometry>
@@ -340,5 +340,5 @@
 		</collision>
 	</xacro:macro>
-	<xacro:macro name="xacro:insert_visu_r_wrist">
+	<xacro:macro name="insert_visu_r_wrist">
 		<visual>
 			<geometry>
@@ -354,5 +354,5 @@
 		</collision>
 	</xacro:macro>
-	<xacro:macro name="xacro:insert_visu_LForeArm">
+	<xacro:macro name="insert_visu_LForeArm">
 		<visual>
 			<geometry>
@@ -368,5 +368,5 @@
 		</collision>
 	</xacro:macro>
-	<xacro:macro name="xacro:insert_visu_LThumb2_link">
+	<xacro:macro name="insert_visu_LThumb2_link">
 		<visual>
 			<geometry>
@@ -382,5 +382,5 @@
 		</collision>
 	</xacro:macro>
-	<xacro:macro name="xacro:insert_visu_LFinger12_link">
+	<xacro:macro name="insert_visu_LFinger12_link">
 		<visual>
 			<geometry>
@@ -396,5 +396,5 @@
 		</collision>
 	</xacro:macro>
-	<xacro:macro name="xacro:insert_visu_RShoulder">
+	<xacro:macro name="insert_visu_RShoulder">
 		<visual>
 			<geometry>
@@ -410,5 +410,5 @@
 		</collision>
 	</xacro:macro>
-	<xacro:macro name="xacro:insert_visu_RFinger23_link">
+	<xacro:macro name="insert_visu_RFinger23_link">
 		<visual>
 			<geometry>
@@ -424,5 +424,5 @@
 		</collision>
 	</xacro:macro>
-	<xacro:macro name="xacro:insert_visu_l_wrist">
+	<xacro:macro name="insert_visu_l_wrist">
 		<visual>
 			<geometry>
@@ -438,5 +438,5 @@
 		</collision>
 	</xacro:macro>
-	<xacro:macro name="xacro:insert_visu_RBicep">
+	<xacro:macro name="insert_visu_RBicep">
 		<visual>
 			<geometry>
@@ -452,5 +452,5 @@
 		</collision>
 	</xacro:macro>
-	<xacro:macro name="xacro:insert_visu_WheelB_link">
+	<xacro:macro name="insert_visu_WheelB_link">
 		<visual>
 			<geometry>
@@ -466,5 +466,5 @@
 		</collision>
 	</xacro:macro>
-	<xacro:macro name="xacro:insert_visu_LFinger23_link">
+	<xacro:macro name="insert_visu_LFinger23_link">
 		<visual>
 			<geometry>
@@ -480,5 +480,5 @@
 		</collision>
 	</xacro:macro>
-	<xacro:macro name="xacro:insert_visu_RElbow">
+	<xacro:macro name="insert_visu_RElbow">
 		<visual>
 			<geometry>
@@ -494,5 +494,5 @@
 		</collision>
 	</xacro:macro>
-	<xacro:macro name="xacro:insert_visu_Neck">
+	<xacro:macro name="insert_visu_Neck">
 		<visual>
 			<geometry>
@@ -508,5 +508,5 @@
 		</collision>
 	</xacro:macro>
-	<xacro:macro name="xacro:insert_visu_LFinger43_link">
+	<xacro:macro name="insert_visu_LFinger43_link">
 		<visual>
 			<geometry>
@@ -522,5 +522,5 @@
 		</collision>
 	</xacro:macro>
-	<xacro:macro name="xacro:insert_visu_RFinger43_link">
+	<xacro:macro name="insert_visu_RFinger43_link">
 		<visual>
 			<geometry>
@@ -536,5 +536,5 @@
 		</collision>
 	</xacro:macro>
-	<xacro:macro name="xacro:insert_visu_torso">
+	<xacro:macro name="insert_visu_torso">
 		<visual>
 			<geometry>
@@ -550,5 +550,5 @@
 		</collision>
 	</xacro:macro>
-	<xacro:macro name="xacro:insert_visu_RFinger42_link">
+	<xacro:macro name="insert_visu_RFinger42_link">
 		<visual>
 			<geometry>
@@ -564,5 +564,5 @@
 		</collision>
 	</xacro:macro>
-	<xacro:macro name="xacro:insert_visu_LFinger31_link">
+	<xacro:macro name="insert_visu_LFinger31_link">
 		<visual>
 			<geometry>
@@ -578,5 +578,5 @@
 		</collision>
 	</xacro:macro>
-	<xacro:macro name="xacro:insert_visu_RFinger33_link">
+	<xacro:macro name="insert_visu_RFinger33_link">
 		<visual>
 			<geometry>
@@ -592,5 +592,5 @@
 		</collision>
 	</xacro:macro>
-	<xacro:macro name="xacro:insert_visu_RForeArm">
+	<xacro:macro name="insert_visu_RForeArm">
 		<visual>
 			<geometry>
@@ -606,5 +606,5 @@
 		</collision>
 	</xacro:macro>
-	<xacro:macro name="xacro:insert_visu_WheelFL_link">
+	<xacro:macro name="insert_visu_WheelFL_link">
 		<visual>
 			<geometry>
@@ -620,5 +620,5 @@
 		</collision>
 	</xacro:macro>
-	<xacro:macro name="xacro:insert_visu_WheelFR_link">
+	<xacro:macro name="insert_visu_WheelFR_link">
 		<visual>
 			<geometry>
@@ -634,5 +634,5 @@
 		</collision>
 	</xacro:macro>
-	<xacro:macro name="xacro:insert_visu_LShoulder">
+	<xacro:macro name="insert_visu_LShoulder">
 		<visual>
 			<geometry>
@@ -648,5 +648,5 @@
 		</collision>
 	</xacro:macro>
-	<xacro:macro name="xacro:insert_visu_Pelvis">
+	<xacro:macro name="insert_visu_Pelvis">
 		<visual>
 			<geometry>
