Commit message: adding new grasp frame

File: pepper_description/urdf/pepper1.0_generated_urdf/pepper.urdf (robot description, URDF)
Before this commit: robot JulietteY20MP, 83 links, 82 joints
Links:
- added link l_grasp_link, mass 2e-06
- added link r_grasp_link, mass 2e-06
Joints:
- added joint LGrasp: type revolute, parent l_wrist, child l_grasp_link, origin xyz=0.065 0 0 rpy=0 0 0, limit lower=0.0 upper=0.0 effort=0.0 velocity=0.0
- added joint RGrasp: type revolute, parent r_wrist, child r_grasp_link, origin xyz=0.065 0 0 rpy=0.0 0 0, limit lower=0.0 upper=0.0 effort=0.0 velocity=0.0
- joint LHand: parent l_wrist -> l_grasp_link
- joint RHand: parent r_wrist -> r_grasp_link

File: pepper_description/urdf/pepper1.0_generated_urdf/pepperGazebo.xacro (robot description, xacro)
@@ -48,4 +48,7 @@
         <plugin name="${side_small}_gripper" filename="libroboticsgroup_gazebo_disable_link_plugin.so">
             <link>${side_small}_gripper</link>
+        </plugin>
+        <plugin name="${side_small}_grasp_link" filename="libroboticsgroup_gazebo_disable_link_plugin.so">
+            <link>${side_small}_grasp_link</link>
         </plugin>
     </xacro:macro>
@@ -169,4 +172,10 @@
         <turnGravityOff>false</turnGravityOff>
     </gazebo>
+    <gazebo reference="l_grasp_link">
+        <mu1>0.5</mu1>
+        <mu2>0.5</mu2>
+        <selfCollide>false</selfCollide>
+        <turnGravityOff>false</turnGravityOff>
+    </gazebo>
     <gazebo reference="l_gripper">
         <mu1>0.5</mu1>
@@ -200,4 +209,10 @@
     </gazebo>
     <gazebo reference="r_wrist">
+        <mu1>0.5</mu1>
+        <mu2>0.5</mu2>
+        <selfCollide>false</selfCollide>
+        <turnGravityOff>false</turnGravityOff>
+    </gazebo>
+    <gazebo reference="r_grasp_link">
         <mu1>0.5</mu1>
         <mu2>0.5</mu2>

File: pepper_description/urdf/pepper1.0_generated_urdf/pepperTransmission.xacro (robot description, xacro)
@@ -85,4 +85,14 @@
 			</actuator>
 		</transmission>
+		<transmission name="${side}Grasp_Transmission">
+			<type>transmission_interface/SimpleTransmission</type>
+			<joint name="${side}Grasp">
+				<hardwareInterface>PositionJointInterface</hardwareInterface>
+			</joint>
+			<actuator name="${side}Grasp_Motor">
+				<hardwareInterface>PositionJointInterface</hardwareInterface>
+				<mechanicalReduction>${speed_red_type3B}</mechanicalReduction>
+			</actuator>
+		</transmission>
 		<transmission name="${side}Hand_Transmission">
 			<type>transmission_interface/SimpleTransmission</type>

File: pepper_description/urdf/pepper1.0_generated_urdf/pepper_arms.xacro (robot description, xacro)
@@ -79,6 +79,18 @@
 		<xacro:insert_visu_l_wrist/>
 	</link>
+	<joint name="LGrasp" type="revolute">
+		<parent link="l_wrist"/>
+		<child link="l_grasp_link"/>
+		<origin rpy="0 0 0" xyz="0.065 0 0"/>
+		<limit effort="0.0" lower="0.0" upper="0.0" velocity="0.0"/>
+	</joint>
+	<link name="l_grasp_link">
+		<inertial>
+			<mass value="2e-06"/>
+			<inertia ixx="1.1e-09" ixy="0" ixz="0" iyy="1.1e-09" iyz="0" izz="1.1e-09"/>
+		</inertial>
+	</link>
 	<joint name="LHand" type="revolute">
-		<parent link="l_wrist"/>
+		<parent link="l_grasp_link"/>
 		<child link="l_gripper"/>
 		<origin rpy="0 0 0" xyz="0.025 0 0"/>
@@ -167,6 +179,18 @@
 		<xacro:insert_visu_r_wrist/>
 	</link>
+	<joint name="RGrasp" type="revolute">
+		<parent link="r_wrist"/>
+		<child link="r_grasp_link"/>
+		<origin rpy="0.0 0 0" xyz="0.065 0 0"/>
+		<limit effort="0.0" lower="0.0" upper="0.0" velocity="0.0"/>
+	</joint>
+	<link name="r_grasp_link">
+		<inertial>
+			<mass value="2e-06"/>
+			<inertia ixx="1.1e-09" ixy="0" ixz="0" iyy="1.1e-09" iyz="0" izz="1.1e-09"/>
+		</inertial>
+	</link>
 	<joint name="RHand" type="revolute">
-		<parent link="r_wrist"/>
+		<parent link="r_grasp_link"/>
 		<child link="r_gripper"/>
 		<origin rpy="0 0 0" xyz="0.025 0 0"/>
