Commit message: fix the pepper drifting problem

File: pepper_description/urdf/pepper1.0_generated_urdf/pepper_torso.xacro (robot description, xacro)
@@ -4,4 +4,10 @@
  *********************************************************************-->
 <robot xmlns:xacro="http://www.ros.org/wiki/xacro">
+	<link name="world"/>
+	<joint name="fixed" type="fixed">
+		<parent link="world"/>
+		<child link="base_link"/>
+		<origin rpy="0 0 0" xyz="0 0 0.03"/>
+	</joint>
 	<link name="base_link"/>
 	<joint name="base_link_fixedjoint" type="fixed">

Commit message: Removed link to world

File: pepper_description/urdf/pepper1.0_generated_urdf/pepper_torso.xacro (robot description, xacro)
@@ -4,10 +4,4 @@
  *********************************************************************-->
 <robot xmlns:xacro="http://www.ros.org/wiki/xacro">
-	<link name="world"/>
-	<joint name="fixed" type="fixed">
-		<parent link="world"/>
-		<child link="base_link"/>
-		<origin rpy="0 0 0" xyz="0 0 0.03"/>
-	</joint>
 	<link name="base_link"/>
 	<joint name="base_link_fixedjoint" type="fixed">
